File: transmitter/hardware/pcb/_saved_pcb.sch (KiCad schematic (older format))
At the start: 7 parts, among them SW101 ~RST, X101 Display

Commit message: Work on schematics started
Started the work on the schematics for the transmitter part
Connections:
- net labels added: BL
- net labels removed: BLEN
Changed lines of the file:
@@
 ~RST
 Text Label 4500 3500 0    50   ~ 0
-BLEN
+BL
 Wire Wire Line
 	6950 3600 7000 3600
