File: transmitter/hardware/pcb/ATmega32u4.sch (KiCad schematic (older format))
At the start: 18 parts, among them P201 TestPoint_Alt, P202 TestPoint_Alt, P203 TestPoint_Alt, P204 TestPoint_Alt, Q201 16M, X201 AVR-ISP-6

Commit message: WIP commit
Parts:
- P201, P202, P203, P204: symbol Modules:TestPoint_Alt -> SilentWorks:TestPoint
Changed lines of the file:
@@
 	4200 2250 4200 2350
 $Comp
-L Modules:TestPoint_Alt P?
+L SilentWorks:TestPoint P?
 U 1 1 5D314B0A
 P 4050 3450
@@
 	4050 3450 3700 3450
 $Comp
-L Modules:TestPoint_Alt P?
+L SilentWorks:TestPoint P?
 U 1 1 5D314CB2
 P 4750 3000
@@
 Connection ~ 4750 3000
 $Comp
-L Modules:TestPoint_Alt P?
+L SilentWorks:TestPoint P?
 U 1 1 5D314D5A
 P 4750 3300
@@
 Connection ~ 4750 3300
 $Comp
-L Modules:TestPoint_Alt P?
+L SilentWorks:TestPoint P?
 U 1 1 5D3150EF
 P 4750 4150
