File: transmitter/hardware/pcb/ATmega32u4.sch (KiCad schematic (older format))
At the start: 18 parts, among them P201 TestPoint_Alt, P202 TestPoint_Alt, P203 TestPoint_Alt, P204 TestPoint_Alt, Q201 16M, X201 AVR-ISP-6

Commit message: WIP
Parts:
- renumbered C206 to C201, C207 to C202, C208 to C203, C209 to C204, C202 to C205, C203 to C206, C204 to C207, C201 to C208, C205 to C209, P202 to P201, P203 to P202, P201 to P203, R202 to R201, R201 to R202
Changed lines of the file:
@@
 P 5200 2050
 AR Path="/5CF69126" Ref="C?"  Part="1"
-AR Path="/5CF68CB3/5CF69126" Ref="C206"  Part="1"
-F 0 "C206" H 5315 2096 50  0000 L CNN
+AR Path="/5CF68CB3/5CF69126" Ref="C201"  Part="1"
+F 0 "C201" H 5315 2096 50  0000 L CNN
 F 1 "100n" H 5315 2005 50  0000 L CNN
 F 2 "Capacitor_SMD:C_0603_1608Metric" H 5238 1900 50  0001 C CNN
@@
 P 5500 2050
 AR Path="/5CF6912D" Ref="C?"  Part="1"
-AR Path="/5CF68CB3/5CF6912D" Ref="C207"  Part="1"
-F 0 "C207" H 5615 2096 50  0000 L CNN
+AR Path="/5CF68CB3/5CF6912D" Ref="C202"  Part="1"
+F 0 "C202" H 5615 2096 50  0000 L CNN
 F 1 "100n" H 5615 2005 50  0000 L CNN
 F 2 "Capacitor_SMD:C_0603_1608Metric" H 5538 1900 50  0001 C CNN
@@
 P 5950 2050
 AR Path="/5CF69134" Ref="C?"  Part="1"
-AR Path="/5CF68CB3/5CF69134" Ref="C208"  Part="1"
-F 0 "C208" H 6065 2096 50  0000 L CNN
+AR Path="/5CF68CB3/5CF69134" Ref="C203"  Part="1"
+F 0 "C203" H 6065 2096 50  0000 L CNN
 F 1 "100n" H 6065 2005 50  0000 L CNN
 F 2 "Capacitor_SMD:C_0603_1608Metric" H 5988 1900 50  0001 C CNN
@@
 P 3700 3600
 AR Path="/5CF6915D" Ref="C?"  Part="1"
-AR Path="/5CF68CB3/5CF6915D" Ref="C201"  Part="1"
-F 0 "C201" H 3815 3646 50  0000 L CNN
+AR Path="/5CF68CB3/5CF6915D" Ref="C208"  Part="1"
+F 0 "C208" H 3815 3646 50  0000 L CNN
 F 1 "10n" H 3815 3555 50  0000 L CNN
 F 2 "Capacitor_SMD:C_0603_1608Metric" H 3738 3450 50  0001 C CNN
@@
 P 4750 4350
 AR Path="/5CF69164" Ref="C?"  Part="1"
-AR Path="/5CF68CB3/5CF69164" Ref="C205"  Part="1"
-F 0 "C205" H 4865 4396 50  0000 L CNN
+AR Path="/5CF68CB3/5CF69164" Ref="C209"  Part="1"
+F 0 "C209" H 4865 4396 50  0000 L CNN
 F 1 "1u" H 4865 4305 50  0000 L CNN
 F 2 "Capacitor_SMD:C_0805_2012Metric_Pad1.15x1.40mm_HandSolder" H 4788 4200 50  0001 C CNN
@@
 P 6150 1550
 AR Path="/5CF6917C" Ref="R?"  Part="1"
-AR Path="/5CF68CB3/5CF6917C" Ref="R202"  Part="1"
-F 0 "R202" H 6219 1596 50  0000 L CNN
+AR Path="/5CF68CB3/5CF6917C" Ref="R201"  Part="1"
+F 0 "R201" H 6219 1596 50  0000 L CNN
 F 1 "100R" H 6219 1505 50  0000 L CNN
 F 2 "Resistor_SMD:R_0603_1608Metric" V 6080 1550 50  0001 C CNN
@@
 P 4650 1900
 AR Path="/5CF69193" Ref="R?"  Part="1"
-AR Path="/5CF68CB3/5CF69193" Ref="R201"  Part="1"
-F 0 "R201" H 4581 1946 50  0000 R CNN
+AR Path="/5CF68CB3/5CF69193" Ref="R202"  Part="1"
+F 0 "R202" H 4581 1946 50  0000 R CNN
 F 1 "1k" H 4581 1855 50  0000 R CNN
 F 2 "Resistor_SMD:R_0603_1608Metric" V 4580 1900 50  0001 C CNN
@@
 P 4350 3300
 AR Path="/5CF691B2" Ref="C?"  Part="1"
-AR Path="/5CF68CB3/5CF691B2" Ref="C204"  Part="1"
-F 0 "C204" V 4250 3300 50  0000 C CNN
+AR Path="/5CF68CB3/5CF691B2" Ref="C207"  Part="1"
+F 0 "C207" V 4250 3300 50  0000 C CNN
 F 1 "15p" V 4450 3300 50  0000 C CNN
 F 2 "Capacitor_SMD:C_0603_1608Metric" H 4350 3300 50  0001 C CNN
@@
 P 4350 3000
 AR Path="/5CF691B9" Ref="C?"  Part="1"
-AR Path="/5CF68CB3/5CF691B9" Ref="C203"  Part="1"
-F 0 "C203" V 4250 3000 50  0000 C CNN
+AR Path="/5CF68CB3/5CF691B9" Ref="C206"  Part="1"
+F 0 "C206" V 4250 3000 50  0000 C CNN
 F 1 "15p" V 4450 3000 50  0000 C CNN
 F 2 "Capacitor_SMD:C_0603_1608Metric" H 4350 3000 50  0001 C CNN
@@
 P 4200 2500
 AR Path="/5CFD82AF" Ref="C?"  Part="1"
-AR Path="/5CF68CB3/5CFD82AF" Ref="C202"  Part="1"
-F 0 "C202" H 4315 2546 50  0000 L CNN
+AR Path="/5CF68CB3/5CFD82AF" Ref="C205"  Part="1"
+F 0 "C205" H 4315 2546 50  0000 L CNN
 F 1 "100n" H 4315 2455 50  0000 L CNN
 F 2 "Capacitor_SMD:C_0603_1608Metric" H 4238 2350 50  0001 C CNN
@@
 P 4050 3450
 AR Path="/5D314B0A" Ref="P?"  Part="1"
-AR Path="/5CF68CB3/5D314B0A" Ref="P201"  Part="1"
-F 0 "P201" H 4050 3525 50  0000 C BNN
+AR Path="/5CF68CB3/5D314B0A" Ref="P203"  Part="1"
+F 0 "P203" H 4050 3525 50  0000 C BNN
 F 1 "TestPoint_Alt" H 4325 3475 50  0001 C CNN
 F 2 "TestPoint:TestPoint_Pad_D1.0mm" H 4250 3450 50  0001 C CNN
@@
 P 4750 3000
 AR Path="/5D314CB2" Ref="P?"  Part="1"
-AR Path="/5CF68CB3/5D314CB2" Ref="P202"  Part="1"
-F 0 "P202" H 4775 3050 50  0000 L CNN
+AR Path="/5CF68CB3/5D314CB2" Ref="P201"  Part="1"
+F 0 "P201" H 4775 3050 50  0000 L CNN
 F 1 "TestPoint_Alt" H 5025 3025 50  0001 C CNN
 F 2 "TestPoint:TestPoint_Pad_D1.0mm" H 4950 3000 50  0001 C CNN
@@
 P 4750 3300
 AR Path="/5D314D5A" Ref="P?"  Part="1"
-AR Path="/5CF68CB3/5D314D5A" Ref="P203"  Part="1"
-F 0 "P203" H 4725 3350 50  0000 R CNN
+AR Path="/5CF68CB3/5D314D5A" Ref="P202"  Part="1"
+F 0 "P202" H 4725 3350 50  0000 R CNN
 F 1 "TestPoint_Alt" H 5025 3325 50  0001 C CNN
 F 2 "TestPoint:TestPoint_Pad_D1.0mm" H 4950 3300 50  0001 C CNN
@@
 P 6350 2050
 AR Path="/5D72051F" Ref="C?"  Part="1"
-AR Path="/5CF68CB3/5D72051F" Ref="C209"  Part="1"
-F 0 "C209" H 6465 2096 50  0000 L CNN
+AR Path="/5CF68CB3/5D72051F" Ref="C204"  Part="1"
+F 0 "C204" H 6465 2096 50  0000 L CNN
 F 1 "100n" H 6465 2005 50  0000 L CNN
 F 2 "Capacitor_SMD:C_0603_1608Metric" H 6388 1900 50  0001 C CNN
@@
 Connection ~ 5950 1750
 $Comp
-L power:PWR_FLAG #FLG0101
+L power:PWR_FLAG #FLG0202
 U 1 1 5D7427D1
 P 3850 1500
-F 0 "#FLG0101" H 3850 1575 50  0001 C CNN
+F 0 "#FLG0202" H 3850 1575 50  0001 C CNN
 F 1 "PWR_FLAG" H 3850 1674 50  0000 C CNN
 F 2 "" H 3850 1500 50  0001 C CNN
