File: transmitter/hardware/pcb/pcb.sch (KiCad schematic (older format))
At the start: 75 parts, among them P101 TestPoint_Alt, P102 TestPoint_Alt, P103 TestPoint_Alt, P104 TestPoint_Alt, P105 TestPoint_Alt, P106 TestPoint_Alt, P107 TestPoint_Alt, P108 TestPoint_Alt, P109 TestPoint_Alt, P110 TestPoint_Alt, P111 TestPoint_Alt, P112 TestPoint_Alt, P113 TestPoint_Alt, P114 TestPoint_Alt, P115 TestPoint_Alt, P116 TestPoint_Alt, P117 TestPoint_Alt, P118 TestPoint_Alt, P119 TestPoint_Alt, P120 TestPoint_Alt, P121 TestPoint_Alt, P122 TestPoint_Alt, P123 TestPoint_Alt, P124 TestPoint_Alt, P125 TestPoint_Alt, P126 TestPoint_Alt, P127 TestPoint_Alt, P128 TestPoint_Alt, P129 TestPoint_Alt, P130 TestPoint_Alt, P131 TestPoint_Alt, Q101 BC847, SW101 ~RST, U101 AMS1117-3.3, X101 USB_B_Micro, X102 SW1, X103 SW2, X104 SW3, X105 SW4, X106 SW5, X107 SW6, X108 SW7, X109 SW8, X110 PWR_5V, X111 UART, X112 gimbal_left_h, X113 gimbal_left_v, X114 gimbal_right_h, X115 gimbal_right_v, X116 analog trimm buttons, X117 Display

Commit message: WIP commit
Parts:
- removed C106: 100n, Capacitor_SMD:C_0805_2012Metric_Pad1.15x1.40mm_HandSolder, symbol Device:C
- removed P112, P113, P114, P117, P118: TestPoint_Alt, TestPoint:TestPoint_Pad_D1.0mm, symbol Modules:TestPoint_Alt
- removed R101, R102: 22R, Resistor_SMD:R_0603_1608Metric, symbol Device:R
- removed R103: 2k, Resistor_SMD:R_0603_1608Metric, symbol Device:R
- removed R104, R106: 1k, Resistor_SMD:R_0603_1608Metric, symbol Device:R
- removed R105: 2.9k, Resistor_SMD:R_0603_1608Metric, symbol Device:R
- removed R107: 330R, Resistor_SMD:R_0603_1608Metric, symbol Device:R
- removed R108: 0R, Resistor_SMD:R_0603_1608Metric, symbol Device:R
- removed R109: 6.8k, Resistor_SMD:R_0603_1608Metric, symbol Device:R
- removed R110: 1.6k, Resistor_SMD:R_0603_1608Metric, symbol Device:R
- removed R111: 620R, Resistor_SMD:R_0603_1608Metric, symbol Device:R
- removed R112: 150R, Resistor_SMD:R_0603_1608Metric, symbol Device:R
- removed S102: 74AHC1G125, Package_TO_SOT_SMD:SOT-353_SC-70-5, symbol 74xGxx:74AHC1G125
- removed X101: USB_B_Micro, Connector_USB:USB_Micro-B_GCT_USB3076-30-A, symbol Connector:USB_B_Micro
- removed X111: UART, Connector_PinHeader_2.54mm:PinHeader_1x04_P2.54mm_Vertical, symbol Connector_Generic:Conn_01x04
- removed X116: analog trimm buttons, Connector_PinHeader_2.54mm:PinHeader_1x09_P2.54mm_Vertical, symbol Connector_Generic:Conn_01x09
- added C?: 10u, Capacitor_SMD:C_1206_3216Metric, symbol Device:C
- added C? (x3): 100n, Capacitor_SMD:C_0805_2012Metric_Pad1.15x1.40mm_HandSolder, symbol Device:C
- added P? (x13): TestPoint_Alt, TestPoint:TestPoint_Pad_D1.0mm, symbol SilentWorks:TestPoint
- added R?: 2k, Resistor_SMD:R_0603_1608Metric, symbol Device:R
- added RN?: 1k, Resistor_THT:R_Array_SIP9, symbol Device:R_Network08
- added S?: ProMicro, symbol promicro:ProMicro
- added S?: 74HC165, Package_SO:SOIC-16_3.9x9.9mm_P1.27mm, symbol 74xx:74LS165
- added S?: 74AHC1G125, Package_TO_SOT_SMD:SOT-353_SC-70-5, symbol 74xGxx:74AHC1G125
- added X?: SW2, Connector_PinHeader_2.54mm:PinHeader_1x02_P2.54mm_Vertical, symbol Connector_Generic:Conn_01x02
- added X?: SW3, Connector_PinHeader_2.54mm:PinHeader_1x02_P2.54mm_Vertical, symbol Connector_Generic:Conn_01x02
- added X?: SW4, Connector_PinHeader_2.54mm:PinHeader_1x02_P2.54mm_Vertical, symbol Connector_Generic:Conn_01x02
- added X?: SW5, Connector_PinHeader_2.54mm:PinHeader_1x02_P2.54mm_Vertical, symbol Connector_Generic:Conn_01x02
- added X?: SW6, Connector_PinHeader_2.54mm:PinHeader_1x02_P2.54mm_Vertical, symbol Connector_Generic:Conn_01x02
- added X?: SW7, Connector_PinHeader_2.54mm:PinHeader_1x02_P2.54mm_Vertical, symbol Connector_Generic:Conn_01x02
- added X?: SW8, Connector_PinHeader_2.54mm:PinHeader_1x02_P2.54mm_Vertical, symbol Connector_Generic:Conn_01x02
- added X?: SW1, Connector_PinHeader_2.54mm:PinHeader_1x02_P2.54mm_Vertical, symbol Connector_Generic:Conn_01x02
- added X?: UART, symbol Connector_Generic:Conn_01x04
- P101, P102, P103, P104, P105, P106, P107, P108, P109, P110, P111, P115, P116, P119, P120, P121, P122, P123, P124, P125, P126, P127, P128, P129, P130, P131: symbol Modules:TestPoint_Alt -> SilentWorks:TestPoint
Connections:
- net labels added: NRF24_CE, ~NRF24_CS
- net labels removed: AN_TRIM_BUTTONS, CE, VBUS, ~CE3, ~CS1
- wire segments 267 -> 299
- no-connect marks 3 -> 4
Other:
- moved on the sheet: Q101
