File: transmitter/hardware/pcb/pcb.sch (KiCad schematic (older format))
At the start: 7 parts, among them SW101 ~RST, X101 Display

Commit message: WIP commit
Parts:
- removed S101: nRF24L01+, Arduino:NRF24L01, symbol nRF24L01+:nRF24L01+
- removed S102: SparkFun_Pro_Micro, Arduino:DIP-24_600, symbol Arduino:SparkFun_Pro_Micro
- added C102, C103, C104, C106: 100n, Capacitor_SMD:C_0805_2012Metric_Pad1.15x1.40mm_HandSolder, symbol Device:C
- added C105: 10u, Capacitor_SMD:C_1206_3216Metric, symbol Device:C
- added P101, P102, P103, P104, P105, P106, P107, P108, P109, P110, P111, P112, P113, P114, P115, P116, P117, P118, P119, P120, P121, P122, P123, P124, P125, P126, P127, P128, P129, P130, P131: TestPoint_Alt, TestPoint:TestPoint_Pad_D1.0mm, symbol Modules:TestPoint_Alt
- added Q101: BC847, Package_TO_SOT_SMD:SOT-23, symbol Transistor_BJT:BC847
- added R101, R102: 22R, Resistor_SMD:R_0603_1608Metric, symbol Device:R
- added R103: 2k, Resistor_SMD:R_0603_1608Metric, symbol Device:R
- added R104, R106: 1k, Resistor_SMD:R_0603_1608Metric, symbol Device:R
- added R105: 2.9k, Resistor_SMD:R_0603_1608Metric, symbol Device:R
- added R107: 330R, Resistor_SMD:R_0603_1608Metric, symbol Device:R
- added R108: 0R, Resistor_SMD:R_0603_1608Metric, symbol Device:R
- added R109: 6.8k, Resistor_SMD:R_0603_1608Metric, symbol Device:R
- added R110: 1.6k, Resistor_SMD:R_0603_1608Metric, symbol Device:R
- added R111: 620R, Resistor_SMD:R_0603_1608Metric, symbol Device:R
- added R112: 150R, Resistor_SMD:R_0603_1608Metric, symbol Device:R
- added RN101: 1k, Resistor_THT:R_Array_SIP9, symbol Device:R_Network08
- added S101: 74HC165, Package_SO:SOIC-16_3.9x9.9mm_P1.27mm, symbol 74xx:74LS165
- added S102: 74AHC1G125, Package_TO_SOT_SMD:SOT-353_SC-70-5, symbol 74xGxx:74AHC1G125
- added S103: NRF24L01_Breakout, RF_Module:nRF24L01_Breakout, symbol RF:NRF24L01_Breakout
- added U101: AMS1117-3.3, Package_TO_SOT_SMD:SOT-223-3_TabPin2, symbol Regulator_Linear:AMS1117-3.3
- added X101: USB_B_Micro, Connector_USB:USB_Micro-B_GCT_USB3076-30-A, symbol Connector:USB_B_Micro
- added X102: SW1, Connector_PinHeader_2.54mm:PinHeader_1x02_P2.54mm_Vertical, symbol Connector_Generic:Conn_01x02
- added X103: SW2, Connector_PinHeader_2.54mm:PinHeader_1x02_P2.54mm_Vertical, symbol Connector_Generic:Conn_01x02
- added X104: SW3, Connector_PinHeader_2.54mm:PinHeader_1x02_P2.54mm_Vertical, symbol Connector_Generic:Conn_01x02
- added X105: SW4, Connector_PinHeader_2.54mm:PinHeader_1x02_P2.54mm_Vertical, symbol Connector_Generic:Conn_01x02
- added X106: SW5, Connector_PinHeader_2.54mm:PinHeader_1x02_P2.54mm_Vertical, symbol Connector_Generic:Conn_01x02
- added X107: SW6, Connector_PinHeader_2.54mm:PinHeader_1x02_P2.54mm_Vertical, symbol Connector_Generic:Conn_01x02
- added X108: SW7, Connector_PinHeader_2.54mm:PinHeader_1x02_P2.54mm_Vertical, symbol Connector_Generic:Conn_01x02
- added X109: SW8, Connector_PinHeader_2.54mm:PinHeader_1x02_P2.54mm_Vertical, symbol Connector_Generic:Conn_01x02
- added X110: PWR_5V, Connector_PinHeader_2.54mm:PinHeader_1x02_P2.54mm_Vertical, symbol Connector_Generic:Conn_01x02
- added X111: UART, Connector_PinHeader_2.54mm:PinHeader_1x04_P2.54mm_Vertical, symbol Connector_Generic:Conn_01x04
- added X112: gimbal_left_h, Connector_PinSocket_2.54mm:PinSocket_1x03_P2.54mm_Vertical, symbol Connector_Generic:Conn_01x03
- added X113: gimbal_left_v, Connector_PinSocket_2.54mm:PinSocket_1x03_P2.54mm_Vertical, symbol Connector_Generic:Conn_01x03
- added X114: gimbal_right_h, Connector_PinSocket_2.54mm:PinSocket_1x03_P2.54mm_Vertical, symbol Connector_Generic:Conn_01x03
- added X115: gimbal_right_v, Connector_PinSocket_2.54mm:PinSocket_1x03_P2.54mm_Vertical, symbol Connector_Generic:Conn_01x03
- added X116: analog trimm buttons, Connector_PinHeader_2.54mm:PinHeader_1x09_P2.54mm_Vertical, symbol Connector_Generic:Conn_01x09
- C101: value 100n -> 10u; footprint Capacitor_SMD:C_0805_2012Metric_Pad1.15x1.40mm_HandSolder -> Capacitor_SMD:C_1206_3216Metric
- renumbered C102 to C107, C103 to C108, X101 to X117
Connections:
- net labels added: AN_TRIM_BUTTONS, GIMBAL_LEFT_H, GIMBAL_LEFT_V, GIMBAL_RIGHT_H, GIMBAL_RIGHT_V, LCD_BL, LCD_DC, PE_LATCH, RX, TX, VBUS, ~CE3, ~LCD_CS, ~LCD_RST, ~PE_CS
- net labels removed: AIN1, AIN2, AIN3, AIN4, BLEN, DC, X_LEFT, X_RIGHT, Y_LEFT, Y_RIGHT, ~CS2
- wire segments 58 -> 267
- no-connect marks 1 -> 3

Commit message: WIP
Parts:
- removed P121: TestPoint_Alt, TestPoint:TestPoint_Pad_D1.0mm, symbol Modules:TestPoint_Alt
- added C106, C109, C110, C111: 10u, Capacitor_SMD:C_1206_3216Metric, symbol Device:C
- added C107, C108: 100n, Capacitor_SMD:C_0805_2012Metric_Pad1.15x1.40mm_HandSolder, symbol Device:C
- added D101: green, LED_THT:LED_D3.0mm, symbol Device:LED
- added D102: red, LED_THT:LED_D3.0mm, symbol Device:LED
- added P103, P107, P108, P109, P110, P111, P118, P119, P126, P127, P129, P138, P141, P142, P144: TestPoint_Alt, TestPoint:TestPoint_Pad_D1.0mm, symbol Modules:TestPoint_Alt
- added R101: n.b, Resistor_SMD:R_0603_1608Metric, symbol Device:R
- added R102, R103: 1k, Resistor_SMD:R_0603_1608Metric, symbol Device:R
- added R104: 1,2k, Resistor_SMD:R_0603_1608Metric, symbol Device:R
- added R105: 0R, Resistor_SMD:R_0603_1608Metric, symbol Device:R
- added R106, R107: 4,7k, Resistor_SMD:R_0603_1608Metric, symbol Device:R
- added S101: Step-Up, symbol Modules:Step-Up
- added S103: TP4056, Package_SO:SOIC-8-1EP_3.9x4.9mm_P1.27mm_EP2.35x2.35mm, symbol Modules:TP4056
- added SW101: Power, Module:SW_Graupner_JS202011AQN_DPDT_Angled, symbol Switch:SW_SPDT
- added X102: Charger, Connector_BarrelJack:BarrelJack_Horizontal, symbol Connector:Jack-DC
- added X104: I2C, Connector_PinHeader_2.54mm:PinHeader_1x04_P2.54mm_Vertical, symbol Connector_Generic:Conn_01x04
- added X107: analog_in2, Connector_Molex:Molex_KK-254_AE-6410-05A_1x05_P2.54mm_Vertical, symbol Connector_Generic:Conn_01x05
- added X108: analog_in3, Connector_Molex:Molex_KK-254_AE-6410-05A_1x05_P2.54mm_Vertical, symbol Connector_Generic:Conn_01x05
- added X110: analog_in4, Connector_Molex:Molex_KK-254_AE-6410-05A_1x05_P2.54mm_Vertical, symbol Connector_Generic:Conn_01x05
- added X118: analog_in1, Connector_Molex:Molex_KK-254_AE-6410-05A_1x05_P2.54mm_Vertical, symbol Connector_Generic:Conn_01x05
- X101: renamed from X110; footprint Connector_PinHeader_2.54mm:PinHeader_1x02_P2.54mm_Vertical -> Connector_PinHeader_2.54mm:PinHeader_1x03_P2.54mm_Vertical; symbol Connector_Generic:Conn_01x02 -> Connector_Generic:Conn_01x03
- X109: renamed from X112; footprint Connector_PinSocket_2.54mm:PinSocket_1x03_P2.54mm_Vertical -> Connector_Molex:Molex_KK-254_AE-6410-05A_1x05_P2.54mm_Vertical; symbol Connector_Generic:Conn_01x03 -> Connector_Generic:Conn_01x05
- X111: renamed from X113; footprint Connector_PinSocket_2.54mm:PinSocket_1x03_P2.54mm_Vertical -> Connector_Molex:Molex_KK-254_AE-6410-05A_1x05_P2.54mm_Vertical; symbol Connector_Generic:Conn_01x03 -> Connector_Generic:Conn_01x05
- X112: renamed from X114; footprint Connector_PinSocket_2.54mm:PinSocket_1x03_P2.54mm_Vertical -> Connector_Molex:Molex_KK-254_AE-6410-05A_1x05_P2.54mm_Vertical; symbol Connector_Generic:Conn_01x03 -> Connector_Generic:Conn_01x05
- X115: footprint Connector_PinSocket_2.54mm:PinSocket_1x03_P2.54mm_Vertical -> Connector_Molex:Molex_KK-254_AE-6410-05A_1x05_P2.54mm_Vertical; symbol Connector_Generic:Conn_01x03 -> Connector_Generic:Conn_01x05
- renumbered C104 to C103, C105 to C104, C107 to C105, C108 to C112, C103 to C113, C106 to C114, P115 to P101, P110 to P102, P109 to P104, P120 to P105, P119 to P106, P126 to P112, P129 to P113, P127 to P114, P130 to P115, P128 to P116, P131 to P117, P111 to P120, P118 to P121, P117 to P122, P112 to P123, P114 to P124, P113 to P125, P122 to P128, P123 to P130, P124 to P131, P101 to P132, P102 to P133, P125 to P134, P103 to P135, P116 to P136, P104 to P137, P105 to P139, P106 to P140, P107 to P143, P108 to P145, R101 to R108, R102 to R109, R103 to R110, R109 to R111, R105 to R112, R110 to R113, R106 to R114, R111 to R115, R107 to R116, R112 to R117, R108 to R118, R104 to R119, S103 to S102, S102 to S104, S101 to S105, SW101 to SW102, X117 to X103, X111 to X105, X101 to X106, X102 to X113, X103 to X114, X104 to X116, X105 to X117, X106 to X119, X107 to X120, X108 to X121, X116 to X122, X109 to X123
Connections:
- net labels added: +5C, +BATT, ANALOG_CH1, ANALOG_CH2, ANALOG_CH3, ANALOG_CH4, NTC, SCL, SDA, ~CS_LCD, ~CS_PE, ~CS_nRF24
- net labels removed: IRQ, ~CE3, ~CS1, ~LCD_CS, ~PE_CS
- wire segments 267 -> 373
- no-connect marks 3 -> 5
Other:
- moved on the sheet: Q101, S104, U101
