File: transmitter/hardware/pcb/pcb.sch (KiCad schematic (older format))
At the start: 91 parts, among them M101 MT3608_Modul, P101 TestPoint_Alt, P102 TestPoint_Alt, P103 TestPoint_Alt, P104 TestPoint_Alt, P105 TestPoint_Alt, P106 TestPoint_Alt, P107 TestPoint_Alt, P108 TestPoint_Alt, P109 TestPoint_Alt, P110 TestPoint_Alt, P111 TestPoint_Alt, P112 TestPoint_Alt, P113 TestPoint_Alt, P114 TestPoint_Alt, P115 TestPoint_Alt, P116 TestPoint_Alt, P117 TestPoint_Alt, P118 TestPoint_Alt, P119 TestPoint_Alt, P120 TestPoint_Alt, P121 TestPoint_Alt, P122 TestPoint_Alt, P123 TestPoint_Alt, P124 TestPoint_Alt, P125 TestPoint_Alt, P126 TestPoint_Alt, P127 TestPoint_Alt, P128 TestPoint_Alt, P129 TestPoint_Alt, P130 TestPoint_Alt, P131 TestPoint_Alt, P132 TestPoint_Alt, P133 TestPoint_Alt, P134 TestPoint_Alt, P135 TestPoint_Alt, P136 TestPoint_Alt, P137 TestPoint_Alt, P138 TestPoint_Alt, P139 TestPoint_Alt, P140 TestPoint_Alt, P141 TestPoint_Alt, Q101 BC847, SW101 POWER, SW102 ~RST, X101 power, X102 Display, X103 UART, X104 gimbal_left_h, X105 gimbal_left_v, X106 gimbal_right_h, X107 gimbal_right_v, X108 SW1, X109 SW2, X110 SW3, X111 SW4, X112 SW5, X113 SW6, X114 SW7, X115 SW8, X116 SW1, X117 SW2, X118 SW3, X119 SW4, X120 SW5, X121 SW6, X122 SW7, X123 SW8

Commit message: WIP
Parts:
- removed RN101, RN102: 1k, Resistor_THT:R_Array_SIP9, symbol Device:R_Network08
- removed X108, X116: SW1, Connector_PinHeader_2.54mm:PinHeader_1x02_P2.54mm_Vertical, symbol Connector_Generic:Conn_01x02
- removed X109, X117: SW2, Connector_PinHeader_2.54mm:PinHeader_1x02_P2.54mm_Vertical, symbol Connector_Generic:Conn_01x02
- removed X110, X118: SW3, Connector_PinHeader_2.54mm:PinHeader_1x02_P2.54mm_Vertical, symbol Connector_Generic:Conn_01x02
- removed X111, X119: SW4, Connector_PinHeader_2.54mm:PinHeader_1x02_P2.54mm_Vertical, symbol Connector_Generic:Conn_01x02
- removed X112, X120: SW5, Connector_PinHeader_2.54mm:PinHeader_1x02_P2.54mm_Vertical, symbol Connector_Generic:Conn_01x02
- removed X113, X121: SW6, Connector_PinHeader_2.54mm:PinHeader_1x02_P2.54mm_Vertical, symbol Connector_Generic:Conn_01x02
- removed X114, X122: SW7, Connector_PinHeader_2.54mm:PinHeader_1x02_P2.54mm_Vertical, symbol Connector_Generic:Conn_01x02
- removed X115, X123: SW8, Connector_PinHeader_2.54mm:PinHeader_1x02_P2.54mm_Vertical, symbol Connector_Generic:Conn_01x02
- added R104, R105, R106, R107, R108, R109, R110, R111, R112, R113, R114, R115, R116, R117, R118, R119: 1k, Resistor_SMD:R_0603_1608Metric, symbol Device:R
- added X108: switches_1, Connector_PinHeader_2.54mm:PinHeader_2x08_P2.54mm_Vertical, symbol Connector_Generic:Conn_02x08_Odd_Even
- added X109: switches_2, Connector_PinHeader_2.54mm:PinHeader_2x08_P2.54mm_Vertical, symbol Connector_Generic:Conn_02x08_Odd_Even
Connections:
- wire segments 314 -> 296
Other:
- moved on the sheet: S105

Commit message: add dc jack for charger connection
Parts:
- added X110: chrg_out, Connector_Wire:SolderWirePad_1x01_Drill1.2mm, symbol Connector_Generic:Conn_01x01
- added XA02: charge, Connector_BarrelJack:BarrelJack_Horizontal, symbol Connector:Barrel_Jack
Connections:
- net labels added: +5C
- wire segments 296 -> 301
Changed lines of the file:
@@
 Wire Wire Line
 	3400 13300 4200 13300
+$Comp
+L Connector:Barrel_Jack XA02
+U 1 1 5CFCAC55
+P 1350 3500
+F 0 "XA02" H 1350 3700 50  0000 C CNN
+F 1 "charge" H 1350 3300 50  0000 C CNN
+F 2 "Connector_BarrelJack:BarrelJack_Horizontal" H 1400 3460 50  0001 C CNN
+F 3 "~" H 1400 3460 50  0001 C CNN
+	1    1350 3500
+	1    0    0    -1
+$EndComp
+$Comp
+L power:GND #PWR0136
+U 1 1 5CFCB0ED
+P 1750 3650
+F 0 "#PWR0136" H 1750 3400 50  0001 C CNN
+F 1 "GND" H 1755 3477 50  0000 C CNN
+F 2 "" H 1750 3650 50  0001 C CNN
+F 3 "" H 1750 3650 50  0001 C CNN
+	1    1750 3650
+	1    0    0    -1
+$EndComp
+Wire Wire Line
+	1650 3600 1750 3600
+Wire Wire Line
+	1750 3600 1750 3650
+Wire Wire Line
+	1650 3400 1750 3400
+Wire Wire Line
+	1750 3400 1750 3300
+$Comp
+L power:+5C #PWR0135
+U 1 1 5D009547
+P 1750 3300
+F 0 "#PWR0135" H 1750 3150 50  0001 C CNN
+F 1 "+5C" H 1765 3473 50  0000 C CNN
+F 2 "" H 1750 3300 50  0001 C CNN
+F 3 "" H 1750 3300 50  0001 C CNN
+	1    1750 3300
+	1    0    0    -1
+$EndComp
+Wire Wire Line
+	1750 3400 1900 3400
+Connection ~ 1750 3400
+$Comp
+L Connector_Generic:Conn_01x01 X110
+U 1 1 5D04821E
+P 2100 3400
+F 0 "X110" H 2180 3442 50  0000 L CNN
+F 1 "chrg_out" H 2180 3351 50  0000 L CNN
+F 2 "Connector_Wire:SolderWirePad_1x01_Drill1.2mm" H 2100 3400 50  0001 C CNN
+F 3 "~" H 2100 3400 50  0001 C CNN
+	1    2100 3400
+	1    0    0    -1
+$EndComp
 $EndSCHEMATC
