File: transmitter/hardware/pcb/Mega_2560_core_2.2_PM/OpenAVRc_I2C.sch (KiCad schematic (older format))
At the start: 8 parts

Commit message: WIP commit
Parts:
- BT501: renamed from BT?; footprint (none) -> Battery:BatteryHolder_Keystone_1060_1x2032
- C501, C502: renamed from C?; footprint (none) -> Capacitor_SMD:C_0603_1608Metric
- R501, R502: renamed from R?; footprint (none) -> Resistor_SMD:R_0603_1608Metric
- S502: renamed from S?; footprint (none) -> Package_SO:SOIC-8_3.9x4.9mm_P1.27mm
- X501: renamed from X?; footprint (none) -> Connector_PinSocket_2.54mm:PinSocket_1x04_P2.54mm_Vertical
- gave numbers to parts that had none: 1
Changed lines of the file:
@@
 $Descr A4 11693 8268
 encoding utf-8
-Sheet 5 5
+Sheet 5 9
 Title ""
 Date ""
@@
 $EndDescr
 $Comp
-L Timer_RTC:DS3231MZ S?
+L Timer_RTC:DS3231MZ S501
 U 1 1 5D752B2C
 P 3400 2950
-F 0 "S?" H 3050 3300 50  0000 C CNN
+F 0 "S501" H 3050 3300 50  0000 C CNN
 F 1 "DS3231MZ" H 3100 2600 50  0000 C CNN
 F 2 "Package_SO:SOIC-8_3.9x4.9mm_P1.27mm" H 3400 2450 50  0001 C CNN
@@
 $EndComp
 $Comp
-L power:GND #PWR?
+L power:GND #PWR0505
 U 1 1 5D7534E3
 P 3400 3350
-F 0 "#PWR?" H 3400 3100 50  0001 C CNN
+F 0 "#PWR0505" H 3400 3100 50  0001 C CNN
 F 1 "GND" H 3405 3177 50  0000 C CNN
 F 2 "" H 3400 3350 50  0001 C CNN
@@
 $EndComp
 $Comp
-L power:+5V #PWR?
+L power:+5V #PWR0501
 U 1 1 5D753A32
 P 3400 2000
-F 0 "#PWR?" H 3400 1850 50  0001 C CNN
+F 0 "#PWR0501" H 3400 1850 50  0001 C CNN
 F 1 "+5V" H 3415 2173 50  0000 C CNN
 F 2 "" H 3400 2000 50  0001 C CNN
@@
 	3400 2000 3400 2050
 $Comp
-L Device:C C?
+L Device:C C501
 U 1 1 5D754085
 P 3550 2200
-F 0 "C?" H 3665 2246 50  0000 L CNN
+F 0 "C501" H 3665 2246 50  0000 L CNN
 F 1 "100n" H 3665 2155 50  0000 L CNN
-F 2 "" H 3588 2050 50  0001 C CNN
+F 2 "Capacitor_SMD:C_0603_1608Metric" H 3588 2050 50  0001 C CNN
 F 3 "~" H 3550 2200 50  0001 C CNN
 	1    3550 2200
@@
 	3400 2050 3400 2550
 $Comp
-L power:GND #PWR?
+L power:GND #PWR0504
 U 1 1 5D754C78
 P 3550 2350
-F 0 "#PWR?" H 3550 2100 50  0001 C CNN
+F 0 "#PWR0504" H 3550 2100 50  0001 C CNN
 F 1 "GND" H 3555 2177 50  0000 C CNN
 F 2 "" H 3550 2350 50  0001 C CNN
@@
 	3300 2050 3300 2550
 $Comp
-L Device:Battery_Cell BT?
+L Device:Battery_Cell BT501
 U 1 1 5D758094
 P 3150 2250
-F 0 "BT?" H 3250 2350 50  0000 L CNN
+F 0 "BT501" H 3250 2350 50  0000 L CNN
 F 1 "Battery_Cell" H 3250 2250 50  0000 L CNN
-F 2 "" V 3150 2310 50  0001 C CNN
+F 2 "Battery:BatteryHolder_Keystone_1060_1x2032" V 3150 2310 50  0001 C CNN
 F 3 "~" V 3150 2310 50  0001 C CNN
 	1    3150 2250
@@
 $EndComp
 $Comp
-L power:GND #PWR?
+L power:GND #PWR0503
 U 1 1 5D759011
 P 3150 2350
-F 0 "#PWR?" H 3150 2100 50  0001 C CNN
+F 0 "#PWR0503" H 3150 2100 50  0001 C CNN
 F 1 "GND" H 3155 2177 50  0000 C CNN
 F 2 "" H 3150 2350 50  0001 C CNN
@@
 $EndComp
 $Comp
-L Device:R R?
+L Device:R R501
 U 1 1 5D75A75A
 P 4050 2550
-F 0 "R?" H 4100 2600 50  0000 L CNN
+F 0 "R501" H 4100 2600 50  0000 L CNN
 F 1 "10k" H 4100 2500 50  0000 L CNN
-F 2 "" V 3980 2550 50  0001 C CNN
+F 2 "Resistor_SMD:R_0603_1608Metric" V 3980 2550 50  0001 C CNN
 F 3 "~" H 4050 2550 50  0001 C CNN
 	1    4050 2550
@@
 $EndComp
 $Comp
-L Device:R R?
+L Device:R R502
 U 1 1 5D75B124
 P 4250 2550
-F 0 "R?" H 4300 2600 50  0000 L CNN
+F 0 "R502" H 4300 2600 50  0000 L CNN
 F 1 "10k" H 4300 2500 50  0000 L CNN
-F 2 "" V 4180 2550 50  0001 C CNN
+F 2 "Resistor_SMD:R_0603_1608Metric" V 4180 2550 50  0001 C CNN
 F 3 "~" H 4250 2550 50  0001 C CNN
 	1    4250 2550
@@
 $EndComp
 $Comp
-L power:+5V #PWR?
+L power:+5V #PWR0502
 U 1 1 5D75B477
 P 4050 2250
-F 0 "#PWR?" H 4050 2100 50  0001 C CNN
+F 0 "#PWR0502" H 4050 2100 50  0001 C CNN
 F 1 "+5V" H 4065 2423 50  0000 C CNN
 F 2 "" H 4050 2250 50  0001 C CNN
@@
 	2350 2850 2700 2850
 $Comp
-L Memory_EEPROM:24LC32 S?
+L Memory_EEPROM:24LC32 S502
 U 1 1 5D75F82F
 P 3450 4600
-F 0 "S?" H 3200 4850 50  0000 C CNN
+F 0 "S502" H 3200 4850 50  0000 C CNN
 F 1 "24LC32" H 3200 4350 50  0000 C CNN
-F 2 "" H 3450 4600 50  0001 C CNN
+F 2 "Package_SO:SOIC-8_3.9x4.9mm_P1.27mm" H 3450 4600 50  0001 C CNN
 F 3 "http://ww1.microchip.com/downloads/en/DeviceDoc/21072G.pdf" H 3450 4600 50  0001 C CNN
 	1    3450 4600
@@
 $EndComp
 $Comp
-L power:+5V #PWR?
+L power:+5V #PWR0506
 U 1 1 5D761A2E
 P 3450 3900
-F 0 "#PWR?" H 3450 3750 50  0001 C CNN
+F 0 "#PWR0506" H 3450 3750 50  0001 C CNN
 F 1 "+5V" H 3465 4073 50  0000 C CNN
 F 2 "" H 3450 3900 50  0001 C CNN
@@
 	3450 3900 3450 3950
 $Comp
-L Device:C C?
+L Device:C C502
 U 1 1 5D761A35
 P 3950 4100
-F 0 "C?" H 4065 4146 50  0000 L CNN
+F 0 "C502" H 4065 4146 50  0000 L CNN
 F 1 "100n" H 4065 4055 50  0000 L CNN
-F 2 "" H 3988 3950 50  0001 C CNN
+F 2 "Capacitor_SMD:C_0603_1608Metric" H 3988 3950 50  0001 C CNN
 F 3 "~" H 3950 4100 50  0001 C CNN
 	1    3950 4100
@@
 	3450 3950 3450 4300
 $Comp
-L power:GND #PWR?
+L power:GND #PWR0507
 U 1 1 5D761A3E
 P 3950 4250
-F 0 "#PWR?" H 3950 4000 50  0001 C CNN
+F 0 "#PWR0507" H 3950 4000 50  0001 C CNN
 F 1 "GND" H 3955 4077 50  0000 C CNN
 F 2 "" H 3950 4250 50  0001 C CNN
@@
 $EndComp
 $Comp
-L power:GND #PWR?
+L power:GND #PWR0509
 U 1 1 5D761E96
 P 3450 4900
-F 0 "#PWR?" H 3450 4650 50  0001 C CNN
+F 0 "#PWR0509" H 3450 4650 50  0001 C CNN
 F 1 "GND" H 3455 4727 50  0000 C CNN
 F 2 "" H 3450 4900 50  0001 C CNN
@@
 	3950 4700 3950 4900
 $Comp
-L power:GND #PWR?
+L power:GND #PWR0510
 U 1 1 5D762EE4
 P 3950 4900
-F 0 "#PWR?" H 3950 4650 50  0001 C CNN
+F 0 "#PWR0510" H 3950 4650 50  0001 C CNN
 F 1 "GND" H 3955 4727 50  0000 C CNN
 F 2 "" H 3950 4900 50  0001 C CNN
@@
 $EndComp
 $Comp
-L power:GND #PWR?
+L power:GND #PWR0508
 U 1 1 5D7638E4
 P 2950 4900
-F 0 "#PWR?" H 2950 4650 50  0001 C CNN
+F 0 "#PWR0508" H 2950 4650 50  0001 C CNN
 F 1 "GND" H 2955 4727 50  0000 C CNN
 F 2 "" H 2950 4900 50  0001 C CNN
@@
 	2600 2750 2350 2750
 $Comp
-L Connector_Generic:Conn_01x04 X?
+L Connector_Generic:Conn_01x04 X501
 U 1 1 5D76CE39
 P 3300 5600
-F 0 "X?" H 3380 5592 50  0000 L CNN
+F 0 "X501" H 3380 5592 50  0000 L CNN
 F 1 "I2C" H 3380 5501 50  0000 L CNN
-F 2 "" H 3300 5600 50  0001 C CNN
+F 2 "Connector_PinSocket_2.54mm:PinSocket_1x04_P2.54mm_Vertical" H 3300 5600 50  0001 C CNN
 F 3 "~" H 3300 5600 50  0001 C CNN
 	1    3300 5600
@@
 $EndComp
 $Comp
-L power:GND #PWR?
+L power:GND #PWR0512
 U 1 1 5D76D757
 P 3000 5900
-F 0 "#PWR?" H 3000 5650 50  0001 C CNN
+F 0 "#PWR0512" H 3000 5650 50  0001 C CNN
 F 1 "GND" H 3005 5727 50  0000 C CNN
 F 2 "" H 3000 5900 50  0001 C CNN
@@
 	3000 5800 3000 5900
 $Comp
-L power:+5V #PWR?
+L power:+5V #PWR0511
 U 1 1 5D76E27A
 P 3000 5450
-F 0 "#PWR?" H 3000 5300 50  0001 C CNN
+F 0 "#PWR0511" H 3000 5300 50  0001 C CNN
 F 1 "+5V" H 3015 5623 50  0000 C CNN
 F 2 "" H 3000 5450 50  0001 C CNN
