File: transmitter/hardware/pcb/Mega_2560_core_2.2_PM/OpenAVRc_Power.sch (KiCad schematic (older format))
At the start: 25 parts

Commit message: WIP commit
Parts:
- removed D?: LED_Dual_CAC, symbol Device:LED_Dual_CAC
- removed R? (x2): 1k, symbol Device:R_Small
- C201, C203, C204, C207, C208: renamed from C?; footprint (none) -> Capacitor_SMD:C_0603_1608Metric
- C202, C205, C206: renamed from C?; footprint (none) -> Capacitor_SMD:C_1206_3216Metric
- D202: renamed from D?; footprint (none) -> Diode_SMD:D_MicroMELF_Hadsoldering
- L201: renamed from L?; footprint (none) -> Inductor_SMD:L_0603_1608Metric
- M201: renamed from M?; footprint (none) -> Transmitter:MT3608_module
- R203, R204, R205, R206, R207: renamed from R?; footprint (none) -> Resistor_SMD:R_0603_1608Metric
- X201: renamed from X?; footprint (none) -> Connector_Molex:Molex_KK-254_AE-6410-03A_1x03_P2.54mm_Vertical; symbol Connector_Generic:Conn_01x05 -> Connector_Generic:Conn_01x03
- X202, X203: renamed from X?; footprint (none) -> Connector_PinSocket_2.54mm:PinSocket_1x02_P2.54mm_Vertical
- gave numbers to parts that had none: 2
