File: transmitter/hardware/pcb/Mega_2560_core_2.2_PM/OpenAVRc_Sticks.sch (KiCad schematic (older format))
At the start: 64 parts

Commit message: WIP commit
Parts:
- added C314, C315, C316: 100n, Capacitor_SMD:C_0603_1608Metric, symbol Device:C
- added X306: Trim, Connector_PinSocket_2.54mm:PinSocket_1x10_P2.54mm_Vertical, symbol Connector_Generic:Conn_01x10
- added X311: Pot4, Connector_PinSocket_2.54mm:PinSocket_1x03_P2.54mm_Vertical, symbol Connector_Generic:Conn_01x03
- added X313: Pot5, Connector_PinSocket_2.54mm:PinSocket_1x03_P2.54mm_Vertical, symbol Connector_Generic:Conn_01x03
- added X314: Pot6, Connector_PinSocket_2.54mm:PinSocket_1x03_P2.54mm_Vertical, symbol Connector_Generic:Conn_01x03
- C301, C302, C303, C304, C305, C306, C307, C308, C309, C310, C311, C312, C313, C317, C318, C319, C320, C321, C322: renamed from C?; footprint (none) -> Capacitor_SMD:C_0603_1608Metric
- J301, J302, J303, J304: renamed from J?; footprint (none) -> Connector_PinSocket_2.54mm:PinSocket_1x02_P2.54mm_Vertical
- R301, R302, R303, R304, R305, R306, R307, R308, R309, R310, R311, R312, R313, R314: renamed from R?; footprint (none) -> Resistor_SMD:R_0603_1608Metric
- RV301, RV302, RV303, RV304, RV305, RV306, RV307, RV308: renamed from RV?; footprint (none) -> Potentiometer_SMD:Potentiometer_Vishay_TS53YJ_Vertical
- S301: renamed from S?; footprint (none) -> Package_SO:SOIC-14_3.9x8.7mm_P1.27mm
- X301, X302, X305, X307: renamed from X?; footprint (none) -> Connector_Molex:Molex_KK-254_AE-6410-05A_1x05_P2.54mm_Vertical
- X303: renamed from X?; footprint (none) -> Connector_PinSocket_2.54mm:PinSocket_1x10_P2.54mm_Vertical
- X304, X312: renamed from X?; footprint (none) -> Connector_PinSocket_2.54mm:PinSocket_1x06_P2.54mm_Vertical
- X308, X309, X310: renamed from X?; footprint (none) -> Connector_PinSocket_2.54mm:PinSocket_1x03_P2.54mm_Vertical
- X315, X316: renamed from X?; footprint (none) -> Connector_PinSocket_2.54mm:PinSocket_1x04_P2.54mm_Vertical
- gave numbers to parts that had none: 2
Connections:
- net +5VA: now also X311.1 (Pin_1), X313.1 (Pin_1), X314.1 (Pin_1)
- net GND: now also X306.10 (Pin_10), X306.9 (Pin_9)
- net GNDA: now also C314.2, C315.2, C316.2, X311.3 (Pin_3), X313.3 (Pin_3), X314.3 (Pin_3)
- new net Pot4_AN: C314.1, X311.2 (Pin_2)
- new net Pot5_AN: C315.1, X313.2 (Pin_2)
- new net Pot6_AN: C316.1, X314.2 (Pin_2)
- new net SW1: X306.1 (Pin_1)
- new net SW2: X306.2 (Pin_2)
- new net SW3: X306.3 (Pin_3)
- new net SW4: X306.4 (Pin_4)
- new net SW5: X306.5 (Pin_5)
- new net SW6: X306.6 (Pin_6)
- new net SW7: X306.7 (Pin_7)
- new net SW8: X306.8 (Pin_8)
Other:
- moved on the sheet: C310, C312, C313, C317, C318, C319, C320, C321, C322, RN301, RN302, X303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
