File: transmitter/hardware/pcb/Mega_2560_core_2.2_PM/Mega_2560_core_2.2_PM.kicad_pcb (KiCad board)
At the start: 2 copper layers, 131 parts, among them J301 TestPoint_2Pole, J302 TestPoint_2Pole, J303 TestPoint_2Pole, J304 TestPoint_2Pole, J901 Conn_01x04, M201 MT3608_Modul, Q201 Si4532DY, X201 BATT, X202 switch, X203 charge, X301 Stick_RH, X302 Stick_RV, X303 Trim, X304 buttons, X305 Stick_LH, X306 Trim, X307 Stick_LV, X308 Pot1, X309 Pot2, X310 Pot3, X311 Pot4, X312 3-way sw, X313 Pot5, X314 Pot6, X315 encoder 1, X316 encoder 2, X401 AVR-ISP-6, X402 AVR-JTAG-10, X501 I2C, X601 3.5'' LCD, X701 Conn_01x08, X802 USB_OTG, X803 Serial, X901 buzzer, Y401 16MHz

Commit message: WIP
Parts:
- removed X402: AVR-JTAG-10, Connector_IDC:IDC-Header_2x05_P2.54mm_Vertical
- C401, C402, C403, C406, C407: moved to B.Cu
- moved BT501 58.4 mm to (212.2, 112.1)
- moved X401 35.4 mm to (198.1, 34.3), turned to 90 degrees
- moved STP401 31.4 mm to (212.3, 34.2), turned to 180 degrees
- moved C407 29.9 mm to (214.6, 57.1), turned to 180 degrees
- moved C405 29.9 mm to (211.8, 36.2), turned to 90 degrees
- moved C408 28.2 mm to (213.4, 36.2), turned to 270 degrees
- moved R403 28.0 mm to (221.6, 60.3), turned to 90 degrees
- moved C406 27.5 mm to (212.1, 36.8)
- moved C401 20.7 mm to (208.3, 46.4), turned to 90 degrees
- moved C402 20.4 mm to (215.3, 53.3), turned to 180 degrees
- moved C404 19.4 mm to (208.3, 46.4), turned to 90 degrees
- moved R402 18.4 mm to (223.0, 60.3), turned to 270 degrees
- moved C403 16.4 mm to (224.2, 48.3), turned to 270 degrees
Routing:
- net Net-(S401-Pad34): track 0.00 -> 7.83 mm
- net Net-(S401-Pad33): track 0.00 -> 7.38 mm
- net +5V: vias 0 -> 1
