File: transmitter/hardware/pcb/Mega_2560_core_2.2_PM/Mega_2560_core_2.2_PM.sch (KiCad schematic (older format))
At the start: 0 parts

Commit message: WIP
Changed lines of the file:
@@
 F37 "PE2\\AIN0\\XCK0" B R 6700 9800 50
 F38 "PE3\\AIN1\\OC3A" B R 6700 6050 50
-F39 "PE4\\INT4\\OC3B" B R 6700 6400 50
+F39 "PE4\\INT4\\OC3B" B R 6700 9350 50
 F40 "PE5\\INT5\\OC3C" B R 6700 4550 50
 F41 "PE6\\INT6\\T3" B R 6700 9900 50
