File: transmitter/hardware/pcb/Mega_2560_core_2.2_PM/OpenAVRc_Controller.sch (KiCad schematic (older format))
At the start: 16 parts

Commit message: WIP commit
Parts:
- C401, C402, C403, C405, C407, C408: renamed from C?; footprint (none) -> Capacitor_SMD:C_0603_1608Metric
- C404, C406: renamed from C?; footprint (none) -> Capacitor_SMD:C_1206_3216Metric
- R401, R402, R403: renamed from R?; footprint (none) -> Resistor_SMD:R_0603_1608Metric
- STP401: renamed from STP?; footprint (none) -> Resistor_SMD:R_0402_1005Metric
- X401: renamed from X?; footprint (none) -> Connector_IDC:IDC-Header_2x03_P2.54mm_Vertical
- X402: renamed from X?; footprint (none) -> Connector_IDC:IDC-Header_2x05_P2.54mm_Vertical
- Y401: renamed from Y?; footprint (none) -> Crystal:Resonator_SMD_muRata_CSTxExxV-3Pin_3.0x1.1mm_HandSoldering
- gave numbers to parts that had none: 1

Commit message: WIP
Parts:
- removed X402: AVR-JTAG-10, Connector_IDC:IDC-Header_2x05_P2.54mm_Vertical, symbol Connector:AVR-JTAG-10
Connections:
- no-connect marks 2 -> 0
Changed lines of the file:
@@
 Text Label 4950 8100 0    50   ~ 0
 TDI
-$Comp
-L Connector:AVR-JTAG-10 X402
-U 1 1 5D4A6739
-P 1550 10200
-F 0 "X402" H 1170 10246 50  0000 R CNN
-F 1 "AVR-JTAG-10" H 1170 10155 50  0000 R CNN
-F 2 "Connector_IDC:IDC-Header_2x05_P2.54mm_Vertical" V 1400 10350 50  0001 C CNN
-F 3 " ~" H 275 9650 50  0001 C CNN
-	1    1550 10200
-	1    0    0    -1
-$EndComp
-$Comp
-L power:+5V #PWR0418
-U 1 1 5D4AEC36
-P 1450 9500
-F 0 "#PWR0418" H 1450 9350 50  0001 C CNN
-F 1 "+5V" H 1465 9673 50  0000 C CNN
-F 2 "" H 1450 9500 50  0001 C CNN
-F 3 "" H 1450 9500 50  0001 C CNN
-	1    1450 9500
-	1    0    0    -1
-$EndComp
-$Comp
-L power:GND #PWR0419
-U 1 1 5D4BA68D
-P 1550 10800
-F 0 "#PWR0419" H 1550 10550 50  0001 C CNN
-F 1 "GND" H 1555 10627 50  0000 C CNN
-F 2 "" H 1550 10800 50  0001 C CNN
-F 3 "" H 1550 10800 50  0001 C CNN
-	1    1550 10800
-	1    0    0    -1
-$EndComp
-Text Label 2300 9900 2    50   ~ 0
-~RESET
-Wire Wire Line
-	2050 9900 2300 9900
-Wire Wire Line
-	2050 10100 2300 10100
-Wire Wire Line
-	2050 10200 2300 10200
-Wire Wire Line
-	2050 10300 2300 10300
-Wire Wire Line
-	2050 10400 2300 10400
-Text Label 2300 10100 2    50   ~ 0
-TCK
-Text Label 2300 10200 2    50   ~ 0
-TMS
-Text Label 2300 10300 2    50   ~ 0
-TDO
-Text Label 2300 10400 2    50   ~ 0
-TDI
-NoConn ~ 2050 10000
-Wire Wire Line
-	1450 9500 1450 9600
-NoConn ~ 1550 9600
 Text HLabel 3200 7400 0    50   BiDi ~ 0
 PG0
