File: transmitter/hardware/pcb/Mega_32U4_core_1.0/Mega_32U4_core_1.0.kicad_pcb (KiCad board)
At the start: 2 copper layers, 41 parts, among them M101 MT3608 Vout=3.3V, M102 NRF24L01_Breakout, M103 MakerHawkTFT, Q101 Si4532DY, SW101 reset, X101 switch, X102 battery, X103 SPI, X104 AVR-ISP-6, X105 POT1, X106 POT2, X107 mode, X108 Stick_RH, X109 Stick_RV, X110 Stick_LH, X111 Stick_LV, X112 chrg

Commit message: WIP commit
Parts:
- C101: value 100u -> 10u; footprint Capacitor_SMD:CP_Elec_10x10 -> Capacitor_SMD:C_1206_3216Metric; moved to B.Cu
- C102, C103, C104, C106, C107, C108, C109, C110, C111, C112, D101, Q101, R101, R103, R105, R106: moved to B.Cu
- X104: footprint Connector_IDC:IDC-Header_2x03_P2.54mm_Vertical -> Connector_PinSocket_2.54mm:PinSocket_2x03_P2.54mm_Vertical
- X108, X109, X110, X111: footprint Connector_Molex:Molex_KK-254_AE-6410-05A_1x05_P2.54mm_Vertical -> Connector_PinSocket_2.54mm:PinSocket_1x05_P2.54mm_Vertical
- moved M101 102.5 mm to (204.5, 117.5), turned to 180 degrees
- moved C104 98.9 mm to (194.4, 114.3)
- moved X106 91.9 mm to (213.4, 81.3), turned to 180 degrees
- moved X104 90.9 mm to (226.1, 78.7), turned to 270 degrees
- moved C111 90.3 mm to (218.4, 99.1), turned to 270 degrees
- moved C101 85.5 mm to (223.5, 116.8), turned to 270 degrees
- moved C110 84.2 mm to (215.9, 99.1), turned to 270 degrees
- moved R103 80.5 mm to (224.8, 102.9), turned to 180 degrees
- moved C102 80.2 mm to (221.0, 116.8), turned to 270 degrees
- moved X101 79.6 mm to (227.3, 99.1), turned to 180 degrees
- moved X102 74.4 mm to (233.7, 111.8), turned to 90 degrees
- moved D101 74.0 mm to (223.5, 96.5), turned to 90 degrees
- moved C112 72.7 mm to (195.6, 83.8)
- moved C106 70.7 mm to (161.3, 75.1), turned to 270 degrees
- moved C109 67.0 mm to (193.0, 76.2), turned to 270 degrees
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Connections:
- C111 pad 1: /POT2_AN -> GND
- M102 pad 8: (no net) -> Net-(M102-Pad8)
- M103 pad 8: (no net) -> Net-(M103-Pad8)
- S101 pad 24: (no net) -> Net-(S101-Pad24)
- X108 pad 2: (no net) -> Net-(X108-Pad2)
- X108 pad 4: (no net) -> Net-(X108-Pad4)
- X109 pad 2: (no net) -> Net-(X109-Pad2)
- X109 pad 4: (no net) -> Net-(X109-Pad4)
- X110 pad 2: (no net) -> Net-(X110-Pad2)
- X110 pad 4: (no net) -> Net-(X110-Pad4)
- X111 pad 2: (no net) -> Net-(X111-Pad2)
- X111 pad 4: (no net) -> Net-(X111-Pad4)
Routing:
- net GND: track 0.00 -> 211.3 mm
- net +3V3: track 0.00 -> 111.6 mm, vias 0 -> 2
- net /MOSI: track 0.00 -> 27.3 mm
- net /MISO: track 0.00 -> 19.0 mm
- net Net-(Q101-Pad3): track 0.00 -> 18.4 mm
- net /SCK: track 0.00 -> 16.1 mm
- net /LCD_DC: track 0.00 -> 15.2 mm
- net +BATT: track 0.00 -> 14.9 mm
- net /Stick_RV_AN: track 0.00 -> 12.9 mm
- net /Stick_RH_AN: track 0.00 -> 12.9 mm
- net /Stick_LV_AN: track 0.00 -> 12.9 mm
- net /Stick_LH_AN: track 0.00 -> 12.9 mm
- net /~RST: track 0.00 -> 8.41 mm
- net /LCD_BL: track 0.00 -> 7.62 mm
- net Net-(Q101-Pad2): track 0.00 -> 5.21 mm
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