File: transmitter/hardware/pcb/Mega_32U4_core_1.0/Mega_32U4_core_1.0.sch (KiCad schematic (older format))
At the start: 37 parts

Commit message: WIP
Parts:
- added C108: 100n, Capacitor_SMD:C_0603_1608Metric, symbol Device:C
- added M103: MakerHawkTFT, Connector_PinSocket_2.54mm:PinSocket_1x09_P2.54mm_Vertical, symbol SilentWorks:MakerHawkTFT
- added X103: SPI, Connector_PinSocket_2.54mm:PinSocket_1x06_P2.54mm_Vertical, symbol Connector_Generic:Conn_01x06
- added X107: mode, Connector_PinSocket_2.54mm:PinSocket_1x02_P2.54mm_Vertical, symbol Connector_Generic:Conn_01x02
- added X112: chrg, Connector_PinSocket_2.54mm:PinSocket_1x02_P2.54mm_Vertical, symbol Connector_Generic:Conn_01x02
- C101: renamed from C?; footprint (none) -> Capacitor_SMD:CP_Elec_10x10
- C102, C103, C105, C107, C109, C110, C111, C112, C113, C114, C115, C116: renamed from C?; footprint (none) -> Capacitor_SMD:C_0603_1608Metric
- C104, C106: renamed from C?; footprint (none) -> Capacitor_SMD:C_1206_3216Metric
- D101: renamed from D?; footprint (none) -> Diode_SMD:D_SMA
- M101: renamed from M?; footprint (none) -> SilentWorks:MT3608_module
- R101, R102, R103, R104, R105, R106: renamed from R?; footprint (none) -> Resistor_SMD:R_0603_1608Metric
- S101: renamed from S?; footprint (none) -> SilentWorks:ProMicro
- SW101: renamed from SW?; footprint (none) -> Button_Switch_THT:SW_PUSH_6mm_H4.3mm
- X101: renamed from X?; footprint (none) -> Connector_PinSocket_2.54mm:PinSocket_1x02_P2.54mm_Vertical
- X102: renamed from X?; footprint (none) -> Connector_Molex:Molex_KK-254_AE-6410-03A_1x03_P2.54mm_Vertical
- X104: renamed from X?; footprint (none) -> Connector_IDC:IDC-Header_2x03_P2.54mm_Vertical
- X105, X106: renamed from X?; footprint (none) -> Connector_PinSocket_2.54mm:PinSocket_1x03_P2.54mm_Vertical
- X108, X109, X110, X111: renamed from X?; footprint (none) -> Connector_Molex:Molex_KK-254_AE-6410-05A_1x05_P2.54mm_Vertical
- gave numbers to parts that had none: 2
Connections:
- net +3V3: now also C108.1, M103.2 (VCC), X103.1 (Pin_1)
- net GND: now also C108.2, M103.1 (GND), X103.6 (Pin_6), X107.2 (Pin_2), X112.2 (Pin_2)
- net MISO: now also X103.4 (Pin_4)
- net MOSI: now also M103.4 (MOSI), X103.3 (Pin_3)
- net PWR_HOLD: now also S101.5 (D0/SCL)
- net SCK: now also M103.3 (SCK), X103.2 (Pin_2)
- net Stick_LH_AN: now also S101.19 (F5); no longer S101.18 (F6)
- net Stick_LV_AN: now also S101.20 (F4); no longer S101.17 (F7)
- net Stick_RH_AN: now also S101.17 (F7); no longer S101.20 (F4)
- net Stick_RV_AN: now also S101.18 (F6); no longer S101.19 (F5)
- net ~nRF_CS: now also M103.5 (MISO)
- net LCD_BL: now reaches S101.1 (D3/TX)
- net LCD_BL: now also M103.9 (BLC)
- net LCD_DC: now reaches S101.2 (D2/RX)
- net LCD_DC: now also M103.7 (DC)
- net ~LCD_CS: now reaches S101.6 (D1/SDA)
- net ~LCD_CS: now also M103.6 (~CS)
- net ~EXP_CS: now reaches S101.7 (D4)
- net ~EXP_CS: now also X103.5 (Pin_5)
- net MODE_SW: now reaches S101.9 (D7)
- net MODE_SW: now also X107.1 (Pin_1)
- net at X102.3 (Pin_3): now also X112.1 (Pin_1)
Other:
- moved on the sheet: C101, C102, C103, C104, C105, C106, C107, C109, C110, C111, C112, C113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

Commit message: WIP commit
Parts:
- removed C101: 100u, Capacitor_SMD:CP_Elec_10x10, symbol Device:CP
- added C101: 10u, Capacitor_SMD:C_1206_3216Metric, symbol Device:C
- X104: footprint Connector_IDC:IDC-Header_2x03_P2.54mm_Vertical -> Connector_PinSocket_2.54mm:PinSocket_2x03_P2.54mm_Vertical
- X108, X109, X110, X111: footprint Connector_Molex:Molex_KK-254_AE-6410-05A_1x05_P2.54mm_Vertical -> Connector_PinSocket_2.54mm:PinSocket_1x05_P2.54mm_Vertical
Connections:
- net +BATT: now also C101.1
- net GND: now also C111.1, C101.2
- net POT2_AN: no longer C111.1
Changed lines of the file:
@@
 Wire Wire Line
 	3850 850  3850 900
-Wire Wire Line
-	3850 850  4900 850
 Connection ~ 3850 850
 Wire Wire Line
@@
 Text GLabel 4300 1250 2    50   Output ~ 0
 VBAT_AN
-$Comp
-L Device:CP C101
-U 1 1 5D1C7412
-P 4900 1050
-F 0 "C101" H 5018 1096 50  0000 L CNN
-F 1 "100u" H 5018 1005 50  0000 L CNN
-F 2 "Capacitor_SMD:CP_Elec_10x10" H 4938 900 50  0001 C CNN
-F 3 "~" H 4900 1050 50  0001 C CNN
-	1    4900 1050
-	1    0    0    -1
-$EndComp
 $Comp
 L Device:C C102
@@
 	1    0    0    -1
 $EndComp
-Wire Wire Line
-	4900 900  4900 850
-Connection ~ 4900 850
-Wire Wire Line
-	4900 850  5300 850
-Wire Wire Line
-	4900 1200 4900 1250
-Wire Wire Line
-	4900 1250 5300 1250
 Connection ~ 5300 1250
 Wire Wire Line
@@
 F 0 "X108" H 1230 8742 50  0000 L CNN
 F 1 "Stick_RH" H 1230 8651 50  0000 L CNN
-F 2 "Connector_Molex:Molex_KK-254_AE-6410-05A_1x05_P2.54mm_Vertical" H 1150 8700 50  0001 C CNN
+F 2 "Connector_PinSocket_2.54mm:PinSocket_1x05_P2.54mm_Vertical" H 1150 8700 50  0001 C CNN
 F 3 "~" H 1150 8700 50  0001 C CNN
 	1    1150 8700
@@
 F 0 "X109" H 1230 9292 50  0000 L CNN
 F 1 "Stick_RV" H 1230 9201 50  0000 L CNN
-F 2 "Connector_Molex:Molex_KK-254_AE-6410-05A_1x05_P2.54mm_Vertical" H 1150 9250 50  0001 C CNN
+F 2 "Connector_PinSocket_2.54mm:PinSocket_1x05_P2.54mm_Vertical" H 1150 9250 50  0001 C CNN
 F 3 "~" H 1150 9250 50  0001 C CNN
 	1    1150 9250
@@
 F 0 "X111" H 1230 10392 50  0000 L CNN
 F 1 "Stick_LV" H 1230 10301 50  0000 L CNN
-F 2 "Connector_Molex:Molex_KK-254_AE-6410-05A_1x05_P2.54mm_Vertical" H 1150 10350 50  0001 C CNN
+F 2 "Connector_PinSocket_2.54mm:PinSocket_1x05_P2.54mm_Vertical" H 1150 10350 50  0001 C CNN
 F 3 "~" H 1150 10350 50  0001 C CNN
 	1    1150 10350
@@
 F 0 "X110" H 1230 9842 50  0000 L CNN
 F 1 "Stick_LH" H 1230 9751 50  0000 L CNN
-F 2 "Connector_Molex:Molex_KK-254_AE-6410-05A_1x05_P2.54mm_Vertical" H 1150 9800 50  0001 C CNN
+F 2 "Connector_PinSocket_2.54mm:PinSocket_1x05_P2.54mm_Vertical" H 1150 9800 50  0001 C CNN
 F 3 "~" H 1150 9800 50  0001 C CNN
 	1    1150 9800
@@
 	6900 7050 6900 7150
 Wire Wire Line
-	6800 7050 6800 6950
-Wire Wire Line
-	6450 6950 6800 6950
-Connection ~ 6800 6950
-Wire Wire Line
-	6800 6950 7050 6950
-Wire Wire Line
 	6450 6950 6350 6950
 Connection ~ 6450 6950
@@
 F 0 "X104" H 6720 5596 50  0000 R CNN
 F 1 "AVR-ISP-6" H 6720 5505 50  0000 R CNN
-F 2 "Connector_IDC:IDC-Header_2x03_P2.54mm_Vertical" V 6750 5550 50  0001 C CNN
+F 2 "Connector_PinSocket_2.54mm:PinSocket_2x03_P2.54mm_Vertical" V 6750 5550 50  0001 C CNN
 F 3 " ~" H 5725 4950 50  0001 C CNN
 	1    7000 5500
@@
 Wire Wire Line
 	1300 1950 1300 2000
+Wire Wire Line
+	6450 6950 7050 6950
+Wire Wire Line
+	6800 7050 6900 7050
+Wire Wire Line
+	3850 850  4950 850
+$Comp
+L Device:C C101
+U 1 1 5D202374
+P 4950 1050
+F 0 "C101" H 5065 1096 50  0000 L CNN
+F 1 "10u" H 5065 1005 50  0000 L CNN
+F 2 "Capacitor_SMD:C_1206_3216Metric" H 4988 900 50  0001 C CNN
+F 3 "~" H 4950 1050 50  0001 C CNN
+	1    4950 1050
+	1    0    0    -1
+$EndComp
+Wire Wire Line
+	5300 1250 4950 1250
+Wire Wire Line
+	4950 1250 4950 1200
+Wire Wire Line
+	4950 900  4950 850
+Connection ~ 4950 850
+Wire Wire Line
+	4950 850  5300 850
 $EndSCHEMATC
